Commit message: add mujoco files and functionality

File: scara_mujoco_description_pkg/urdf/scara_trajectory_controller.xacro (robot description, xacro)
@@ -1,5 +1,5 @@
 <?xml version="1.0"?>
 <robot name="robot_scara" xmlns:xacro="http://ros.org/wiki/xacro" >
-    <xacro:property name="package_name" value="examen_description"/>
+    <xacro:property name="package_name" value="scara_mujoco_description_pkg"/>
     <xacro:include filename="$(find ${package_name})/urdf/scara_urdf.xacro"/>
     <xacro:include filename="$(find ${package_name})/urdf/trajectory_controller.xacro"/>

File: scara_mujoco_description_pkg/urdf/trajectory_controller.xacro (robot description, xacro)
@@ -25,11 +25,9 @@
         </joint>
     </ros2_control>
-    <!--Pluging de control
-    <gazebo>
-        <plugin filename="libgazebo_ros2_control.so" name="gazebo_ros2_control" >
-            <robot_param>robot_description</robot_param>
-            <robot_param_node>robot_state_publisher</robot_param_node>
-            <parameters>$(find ${package_name})/config/scara_trajectory_controller.yaml</parameters>
-        </plugin>
-    </gazebo>   -->
+    <!--Pluging de control-->
+    <plugin name="control_plugin" filename="libmujoco_system_plugins.so" >
+        <robot_param>robot_description</robot_param>
+        <robot_param_node>robot_state_publisher</robot_param_node>
+        <parameters>$(find ${package_name})/config/scara_trajectory_controller.yaml</parameters>
+    </plugin>
 </robot>
