Commit message: edit mujoco_models and urdf file to complain with mujoco

File: scara_mujoco_description_pkg/urdf/scara_urdf.xacro (robot description, xacro)
@@ -1,8 +1,8 @@
 <?xml version="1.0" encoding="utf-8"?>
 <robot name="robot_scara" xmlns:xacro="http://ros.org/wiki/xacro">
-    <link name="world">
+    <link name="world_link">
     </link>
     <joint name="world_joint" type="fixed">
-        <parent link="world"/>
+        <parent link="world_link"/>
         <child link="base_link"/>
         <origin xyz="0.0 0 0.0" rpy="0 0 0"/>
